File: hardware/kicad_project/pokey-watch.kicad_pcb (KiCad board)
At the start: 2 copper layers, 46 x 46 mm, 41 parts, among them CON1 USB-MINI-B, K1 CONN_3, P1 CONN_2, P2 CONN_2, SW1 SW_PUSH_SMALL, SW2 SW_PUSH_SMALL, SW3 SWITCH_INV, U1 MCP73831, U2 LPC1313_LQFP48, U3 LM3671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

Commit message: Updated schematic with real net names for the program and reset pins; changed picth-detection algorithm to average 5 points of the FFT for improved accuracy.
Parts:
- R11: value Rfb -> 5.1k
- R12: value 2Rfb -> 340k
Connections:
- net N-0000028 renamed RESET
- net N-0000029 renamed PGRM
